File: switch-n2.kicad_pcb (KiCad board)
At the start: 2 copper layers, 50 x 80 mm, 43 parts, among them J1 61000821121, Q1 ZXMP10A13F, Q2 FDMT80080DC, Q3 FDMT80080DC, Q4 FDMT80080DC, Q5 FDMT80080DC, U1 BQ76200

Commit message: Fixed some comments on schematic
Parts:
- C3: value 4.7u -> 2.2u
- Q2, Q3, Q4, Q5: value FDMT80080DC -> NVMFS6H800NT1G
- R11, R12, R13, R14: value 3m -> 2m

Commit message: Clean up schematics and add pdf version
Parts:
- C3: value 2.2u -> 4.7u
Changed lines of the file:
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@@
       (effects (font (size 1 1) (thickness 0.15)))
     )
-    (fp_text value 2.2u (at 0 1.65 90) (layer F.Fab)
+    (fp_text value 4.7u (at 0 1.65 90) (layer F.Fab)
       (effects (font (size 1 1) (thickness 0.15)))
     )
